File: bowelProbe.kicad_sch (KiCad schematic)
At the start: 27 parts, among them J1 Probe, U1 MAX038CPP, U2 OPA2134PA, U3 MCP6002-E/P, U4 TL072ACP

Commit message: Schematic Nearly Finished
Added important decoupling capacitors. Added in all necessary symbols, footprints, 3D files (except for probe and voltages).

To do:
- Determine plan for probe and power pins
- Set up their symbols, footprints, 3D files
- Final schematic review
- Move on to PCB layout and routing
Parts:
- added C10, C11, C8, C9: 10u, BowelProbe:Capacitor-10u, symbol Device:C_Polarized_Small_US
- added C12, C14, C15, C16, C17: 0.1u, BowelProbe:Capacitor-10n, symbol Device:C_Small
- added C13: 1u, BowelProbe:Capacitor-10n, symbol Device:C_Small
- added C7: 10n, BowelProbe:Capacitor-10n, symbol Device:C_Small
- added D2, D3: 1N5817, BowelProbe:1N5817, symbol Diode:1N4001
- added R15: 1k, BowelProbe:Resistor-20k, symbol Device:R_US
- C1: footprint (none) -> BowelProbe:Capacitor-10n; Order (none) -> https://www.digikey.com/en/products/detail/kemet/C320C104K5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
- C2: value 20n -> 10n; footprint (none) -> BowelProbe:Capacitor-10n; Order (none) -> https://www.digikey.com/en/products/detail/kemet/C322C103J5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
- C3, C6: value 1u -> 1n; footprint (none) -> BowelProbe:Capacitor-10n; Order (none) -> https://www.digikey.com/en/products/detail/kemet/C315C102M1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
- C4, C5: value 1n -> 1u; footprint (none) -> BowelProbe:Capacitor-10n; Order (none) -> https://www.digikey.com/en/products/detail/kemet/C330C105M5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
- R1: footprint (none) -> BowelProbe:Resistor-20k; Order (none) -> https://www.digikey.com/en/products/detail/yageo/MFR100FTF5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
- R10, R11, R12, R13, R14, R4, R5, R6, R7, R8, R9: footprint (none) -> BowelProbe:Resistor-20k; Order (none) -> https://www.digikey.com/en/products/detail/yageo/MFR-25FRF5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
- R2: footprint (none) -> BowelProbe:Resistor-20k; Order (none) -> https://www.digikey.com/en/products/detail/yageo/MFR-25FTF5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
- R3: footprint (none) -> BowelProbe:Resistor-20k; Order (none) -> https://www.digikey.com/en/products/detail/vishay-dale/RN60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
- U1: footprint (none) -> BowelProbe:MAX038CPP
Connections:
- net (LSB): now also A1.16 (D13); no longer A1.13 (D10)
- net (MSB): now also A1.13 (D10); no longer A1.16 (D13)
- net +12V: now also C11.1, C14.2, C16.2
- net +5V: now also C10.1, C12.2, C13.2, D3.1 (K)
- net -12V: now also C15.2, C17.1, C9.2
- net -5V: now also C8.2
- net GND: now also C10.2, C11.2, C12.1, C13.1, C14.1, C15.1, C16.1, C17.2, C7.1, C8.1, C9.1, D2.2 (A)
- net at C1.1, D1.1 (K), R2.1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: now also R15.1; no longer A1.19 (A0)
- net at R12.1, U2.1 (OUT_A), U2.5 (+IN_B): no longer R1.1
- net at U2.6 (-IN_B), U2.7 (OUT_B): now also R1.1
- net at U3.5: now also D2.1 (K), D3.2 (A), R15.2
- net at U3.6: now also A1.19 (A0), U3.7
- net at R8.2: now also A1.15 (D12); no longer A1.14 (D11)
- net at C2.2, U1.5 (COSC): now also C7.2
- net at R6.2: now also A1.14 (D11); no longer A1.15 (D12)
Other:
- note added: "FIGURE OUT FOOTPRINTS: - POWER - PROBE"
- moved on the sheet: A1, C2, R1, R10, R11, R4, R5, R6, R7, R8, R9

Commit message: Schematic and PCB update
Finished schematic. Finished general PCB layout.

To do:
- Finely touch up PCB layout
- Review layout
- Begin routing
Parts:
- removed J1: Probe, symbol Connector:Conn_01x02_Socket
- added J10, J11: Conn_01x01, BowelProbe:CT3149-5, symbol Connector_Generic:Conn_01x01
- added J2, J5, J7, J9: Conn_01x01, BowelProbe:CT3149-2, symbol Connector_Generic:Conn_01x01
- added J3, J4, J6, J8: Conn_01x01, BowelProbe:CT3149-0, symbol Connector_Generic:Conn_01x01
- U2: Order (none) -> https://www.digikey.com/en/products/detail/texas-instrument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
Connections:
- net +12V is gone; now on an unnamed net: C11.1, C14.2, C16.2, U2.8 (V+), U4.8 (VCC+)
- net GND: now also J11.1 (Pin_1), J3.1 (Pin_1), J4.1 (Pin_1), J6.1 (Pin_1), J8.1 (Pin_1)
- net at R1.2, U4.3 (1IN+): now also J10.1 (Pin_1)
- net at A1.30 (VIN): now also J7.1 (Pin_1)
- net (LSB): no longer names the net of A1.16 (D13), R10.2
- net (MSB): no longer names the net of A1.13 (D10), R4.2
- net +5V: no longer names the net of C10.1, C12.2, C13.2, C3.1, C4.1, D3.1 (K), U1.17 (V+), U1.4 (A1), U3.8
- net +5V: now also J9.1 (Pin_1)
- net -12V: no longer names the net of C15.2, C17.1, C9.2, U2.4 (V-), U4.4 (VCC-)
- net -12V: now also J5.1 (Pin_1)
- net -5V: no longer names the net of C5.2, C6.2, C8.2, U1.20 (V-)
- net -5V: now also J2.1 (Pin_1)
- no-connect marks 26 -> 25
Other:
- note added: "(LSB)"
- note added: "(MSB)"
- note added: "+12V"
- note added: "+5V"
- note added: "-12V"
- note added: "-5V"
- note added: "PROBE"
- note removed: "FIGURE OUT FOOTPRINTS: - POWER - PROBE"
